Commit message: fixed training script

File: Genesis/genesis/assets/urdf/q1/kutta.urdf (robot description, URDF)
Before this commit: robot Q1, 9 links, 8 joints
Links:
- link base_link: mass 20.0 -> 10.0
Joints:
- joint RR_calf_joint: origin xyz=0 0.245452 0.0544472 rpy=3.14159263868863 -1.5707963267949 0 -> xyz=0 0.245452 0.0544472 rpy=0 1.5707963267949 0
